Commit message: manual arm control

File: src/ddori_description/urdf/ddori.urdf (robot description, URDF)
Before this commit: robot ddori, 4 links, 3 joints
Links:
- added link left_back_wheel; visual cylinder length=0.03 radius=0.03
- added link left_front_wheel; visual cylinder length=0.03 radius=0.03
- added link motordrv; visual box size=0.16 .142 .05
- added link right_back_wheel; visual cylinder length=0.03 radius=0.03
- added link right_front_wheel; visual cylinder length=0.03 radius=0.03
- link left_arm: geometry visual box size=0.21 .03 .055
- link right_arm: geometry visual box size=0.21 .03 .055
Joints:
- added joint base_to_motordrv: type fixed, parent base_link, child motordrv, origin xyz=0 0 -0.190
- added joint left_back_wheel_joint: type fixed, parent motordrv, child left_back_wheel, origin xyz=-0.071 -0.095 -0.02 rpy=0 0 0, axis 0 1 0
- added joint left_front_wheel_joint: type fixed, parent motordrv, child left_front_wheel, origin xyz=0.071 -0.095 -0.02 rpy=0 0 0
- added joint right_back_wheel_joint: type fixed, parent motordrv, child right_back_wheel, origin xyz=-0.071 0.095 -0.02 rpy=0 0 0, axis 0 1 0
- added joint right_front_wheel_joint: type fixed, parent motordrv, child right_front_wheel, origin xyz=0.071 0.095 -0.02 rpy=0 0 0
- joint base_to_left_arm: origin xyz=-0.135 0 .13 -> xyz=0 -0.135  .13
- joint base_to_right_arm: origin xyz=0.135 0 .13 -> xyz=0 0.135  .13
